File: hardware/pcb/main_board/main_board.kicad_pcb (KiCad board)
At the start: 2 copper layers, 9 parts, among them J1 AmpSensor, J2 VoltSensor, J3 5V, J4 GND, U1 ESP32-DEVKITC-32D

Commit message: Generated PCB
Parts:
- moved R2 118.1 mm to (36.8, 67.6), turned to 90 degrees
- moved R3 103.6 mm to (49.5, 57.4), turned to -90 degrees
- moved C1 96.0 mm to (58.9, 67.0), turned to -90 degrees
- moved J1 93.5 mm to (69.1, 58.9)
- moved R1 91.3 mm to (62.5, 54.6), turned to 180 degrees
- moved U1 81.9 mm to (62.8, 90.2), turned to -90 degrees
- moved J4 78.7 mm to (94.2, 97.5)
- moved J3 77.5 mm to (94.2, 91.9)
- moved J2 74.7 mm to (94.2, 82.5)
Routing:
- net GND: track 0.00 -> 118.2 mm
- net VCC: track 0.00 -> 76.1 mm
- net Net-(C1-Pad1): track 0.00 -> 47.6 mm
- net Net-(U1-IO34): track 0.00 -> 34.3 mm
- net Net-(J2-Pin_1): track 0.00 -> 27.8 mm
- added copper zone on B.Cu, net GND
- added copper zone on F.Cu, net GND
Other:
- board outline added: 69 x 75 mm
- board text added: "GoComputing"
- board text added: "R"
- board text added: "S"
- board text added: "T"
